File: rotor.kicad_pcb (KiCad board)
At the start: 2 copper layers, 100 x 135 mm, 57 parts, among them J1 Power, J10 Analog, J11 Communication, J12 PWM, J13 PWM, J14 Conn_01x16, J15 Conn_01x16, J16 EL_Relay, J17 Conn_01x02, J18 Conn_01x06, J19 Conn_01x02, J2 PWM, J20 LCD 4x16//, J21 Conn_01x04, J22 Push_button_CW, J23 Push_button_CCW, J24 Push_button_UP, J25 Push_button_DwN, J26 AZ_Relay, J29 Conn_01x02, J3 Analog, J30 Nextion, J31 Conn_01x02, J32 Conn_01x02, J33 LCD 4x16 I2C, J34 Conn_01x02, J35 GPS Neo7M, J36 Conn_01x02, J37 Push_button_DwN, J4 PWM, J5 Analog, J6 Communication, J7 Digital, J8 Analog, J9 Power, U1 uA7805

Commit message: minor fixes, new iBom, RTM version
Parts:
- removed J18: Conn_01x06, Connector_Molex:Molex_KK-254_AE-6410-06A_1x06_P2.54mm_Vertical
- removed J32: Conn_01x02, Connector_Molex:Molex_KK-254_AE-6410-02A_1x02_P2.54mm_Vertical
- added REF**: KiCad-Logo2_5mm_SilkScreen, Symbol:KiCad-Logo2_5mm_SilkScreen, F.Cu at (192.0, -21.0)
- added REF**: OSHW-Logo2_7.3x6mm_SilkScreen, Symbol:OSHW-Logo2_7.3x6mm_SilkScreen, F.Cu at (123.7, -21.2)
- added REF**: OSHW-Logo2_7.3x6mm_SilkScreen, Symbol:OSHW-Logo2_7.3x6mm_SilkScreen, B.Cu at (194.9, -20.4)
- added REF**: KiCad-Logo2_6mm_SilkScreen, Symbol:KiCad-Logo2_6mm_SilkScreen, B.Cu at (196.7, -12.2)
- added RV1: 4k7, Potentiometer_SMD:Potentiometer_Bourns_TC33X_Vertical, F.Cu at (198.2, -10.2)
- J37: value Push_button_DwN -> XT30 connector
- moved J37 5.25 mm to (118.2, 60.8), turned to -90 degrees
Connections:
- C1 pad 2: Net-(J37-Pin_1) -> Net-(J37-Pin_2)
- C4 pad 2: Net-(J37-Pin_1) -> Net-(J37-Pin_2)
- C7 pad 1: Net-(J37-Pin_1) -> Net-(J37-Pin_2)
- J20 pad 2: Net-(J20-Pin_2) -> +5V
- J33 pad 1: GND -> SCL
- J33 pad 2: +5V -> SDA
- J33 pad 3: SDA -> +5V
- J33 pad 4: SCL -> GND
- J37 pad 1: Net-(J37-Pin_1) -> GND
- J37 pad 2: GND -> Net-(J37-Pin_2)
- U1 pad 1: Net-(J37-Pin_1) -> Net-(J37-Pin_2)
Routing:
- net +5V: track 252.9 -> 300.9 mm
- net Net-(J37-Pin_2): track 0.00 -> 46.9 mm
- net Net-(J37-Pin_1): track 46.9 -> 0.00 mm
- net Net-(J20-Pin_3): track 0.00 -> 19.9 mm
- net SCL: track 30.9 -> 34.0 mm
- net SDA: track 35.2 -> 36.0 mm
- net E: track 98.4 -> 97.9 mm
Other:
- board text added: "A-Ref GND 13 12 11 10 9 8 7 6 5 4 3 2 RX 0->"
- board text added: "GND TX RX 5V"
- board text added: "GND Vcc Contrast RS RW E D0 D1 D2 D3 D4 D5 D6 D7 Led+ Led-"
- board text added: "LCD Contrast"
- board text added: "Nextion Serial out"
- board text added: "SCL SDA +5V GND"
- board text added: "TX 0->"
- board text added: "TX RX"
- board text removed: "A-Ref GND 13 12 11 10 9 8 7 6 5 4 3 2 TX 0->1 RX 0->0"
- board text removed: "I2C"
- board text removed: "Nextion Serial"
